Commit message: sync https://www.lejuhub.com/highlydynamic/kuavo-ros-control/commit/162ac3a5d40a6edda606c4330e10bff841dff23d

File: src/kuavo_assets/models/biped_s40/urdf/biped_s40.urdf (robot description, URDF)
Before this commit: robot biped_s40, 46 links, 45 joints
Links:
- link leg_l6_link: geometry collision box size=0.25 0.1 0.04; visual mesh filename=package://kuavo_assets/models/biped_s40/meshes/l_foot_roll.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
- link leg_r6_link: geometry collision box size=0.25 0.1 0.04; visual mesh filename=package://kuavo_assets/models/biped_s40/meshes/r_foot_roll.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

File: src/kuavo_assets/models/biped_s40/urdf/drake/biped_v3_arm.urdf (robot description, URDF)
Before this commit: robot biped_v3_arm, 15 links, 14 joints
Links:
- removed link torso
- added link base_link, mass 22.6889; visual mesh filename=../../meshes/base_link.STL
- added link zarm_l7_end_effector; collision sphere radius=0.005
- added link zarm_r7_end_effector; collision sphere radius=0.005
Joints:
- added joint zarm_l7_end_effector_joint: type fixed, parent zarm_l7_link, child zarm_l7_end_effector, origin xyz=0 -0.03 -0.17 rpy=0 0 0
- added joint zarm_r7_end_effector_joint: type fixed, parent zarm_r7_link, child zarm_r7_end_effector, origin xyz=0 0.03 -0.17 rpy=0 0 0
- joint zarm_l1_joint: parent torso -> base_link
- joint zarm_r1_joint: parent torso -> base_link

File: src/kuavo_assets/models/biped_s41/urdf/biped_s41.urdf (robot description, URDF)
Before this commit: robot biped_s41, 46 links, 45 joints
Links:
- link leg_l6_link: geometry collision box size=0.25 0.1 0.04; visual mesh filename=package://kuavo_assets/models/biped_s41/meshes/l_foot_roll.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
- link leg_r6_link: geometry collision box size=0.25 0.1 0.04; visual mesh filename=package://kuavo_assets/models/biped_s41/meshes/r_foot_roll.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

File: src/kuavo_assets/models/biped_s41/urdf/drake/biped_v3_arm.urdf (robot description, URDF)
Before this commit: robot biped_v3_arm, 15 links, 14 joints
Links:
- removed link torso
- added link base_link, mass 23.8489; visual mesh filename=../../meshes/base_link.STL
- added link zarm_l7_end_effector; collision sphere radius=0.005
- added link zarm_r7_end_effector; collision sphere radius=0.005
Joints:
- added joint zarm_l7_end_effector_joint: type fixed, parent zarm_l7_link, child zarm_l7_end_effector, origin xyz=0 -0.03 -0.17 rpy=0 0 0
- added joint zarm_r7_end_effector_joint: type fixed, parent zarm_r7_link, child zarm_r7_end_effector, origin xyz=0 0.03 -0.17 rpy=0 0 0
- joint zarm_l1_joint: parent torso -> base_link
- joint zarm_r1_joint: parent torso -> base_link

File: src/kuavo_assets/models/biped_s42/urdf/biped_s42.urdf (robot description, URDF)
Before this commit: robot biped_s42, 47 links, 46 joints
Links:
- link leg_l6_link: geometry collision box size=0.25 0.1 0.04; visual mesh filename=package://kuavo_assets/models/biped_s42/meshes/l_foot_roll.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
- link leg_r6_link: geometry collision box size=0.25 0.1 0.04; visual mesh filename=package://kuavo_assets/models/biped_s42/meshes/r_foot_roll.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

File: src/kuavo_assets/models/biped_s42/urdf/drake/biped_v3_arm.urdf (robot description, URDF)
Before this commit: robot biped_v3_arm, 15 links, 14 joints
Links:
- removed link torso
- added link base_link, mass 26.30833803; visual mesh filename=../../meshes/torso.STL
- added link zarm_l7_end_effector; collision sphere radius=0.005
- added link zarm_r7_end_effector; collision sphere radius=0.005
Joints:
- added joint zarm_l7_end_effector_joint: type fixed, parent zarm_l7_link, child zarm_l7_end_effector, origin xyz=0 -0.03 -0.17 rpy=0 0 0
- added joint zarm_r7_end_effector_joint: type fixed, parent zarm_r7_link, child zarm_r7_end_effector, origin xyz=0 0.03 -0.17 rpy=0 0 0
- joint zarm_l1_joint: origin xyz=-0.0175 0.25886 0.3245 rpy=0 0 0 -> xyz=-0.017499853 0.26686 0.4245 rpy=0 0 0; parent torso -> base_link
- joint zarm_r1_joint: origin xyz=-0.0175 -0.25886 0.3245 rpy=0 0 0 -> xyz=-0.017499853 -0.26686 0.4245 rpy=0 0 0; parent torso -> base_link

File: src/kuavo_assets/models/biped_s43/urdf/biped_s43.urdf (robot description, URDF)
Before this commit: robot biped_s43, 46 links, 45 joints
Links:
- link leg_l6_link: geometry collision box size=0.25 0.1 0.04; visual mesh filename=package://kuavo_assets/models/biped_s43/meshes/l_foot_roll.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
- link leg_r6_link: geometry collision box size=0.25 0.1 0.04; visual mesh filename=package://kuavo_assets/models/biped_s43/meshes/r_foot_roll.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

File: src/kuavo_assets/models/biped_s43/urdf/drake/biped_v3_arm.urdf (robot description, URDF)
Before this commit: robot biped_v3_arm, 15 links, 14 joints
Links:
- removed link torso
- added link base_link, mass 21.7789; visual mesh filename=../../meshes/base_link.STL
- added link zarm_l7_end_effector; collision sphere radius=0.005
- added link zarm_r7_end_effector; collision sphere radius=0.005
Joints:
- added joint zarm_l7_end_effector_joint: type fixed, parent zarm_l7_link, child zarm_l7_end_effector, origin xyz=0 -0.03 -0.17 rpy=0 0 0
- added joint zarm_r7_end_effector_joint: type fixed, parent zarm_r7_link, child zarm_r7_end_effector, origin xyz=0 0.03 -0.17 rpy=0 0 0
- joint zarm_l1_joint: parent torso -> base_link
- joint zarm_r1_joint: parent torso -> base_link

File: src/kuavo_assets/models/biped_s45/urdf/biped_s45.urdf (robot description, URDF)
Before this commit: robot biped_s45, 47 links, 46 joints
Links:
- link leg_l6_link: geometry collision box size=0.25 0.1 0.04; visual mesh filename=package://kuavo_assets/models/biped_s45/meshes/l_foot_roll.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
- link leg_r6_link: geometry collision box size=0.25 0.1 0.04; visual mesh filename=package://kuavo_assets/models/biped_s45/meshes/r_foot_roll.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

File: src/kuavo_assets/models/biped_s45/urdf/drake/biped_v3_arm.urdf (robot description, URDF)
Before this commit: robot biped_v3_arm, 15 links, 14 joints
Links:
- removed link torso
- added link base_link, mass 22.11293803; visual mesh filename=../../meshes/torso.STL
- added link zarm_l7_end_effector; collision sphere radius=0.005
- added link zarm_r7_end_effector; collision sphere radius=0.005
Joints:
- added joint zarm_l7_end_effector_joint: type fixed, parent zarm_l7_link, child zarm_l7_end_effector, origin xyz=0 -0.03 -0.17 rpy=0 0 0
- added joint zarm_r7_end_effector_joint: type fixed, parent zarm_r7_link, child zarm_r7_end_effector, origin xyz=0 0.03 -0.17 rpy=0 0 0
- joint zarm_l1_joint: parent torso -> base_link
- joint zarm_r1_joint: parent torso -> base_link

File: src/kuavo_assets/models/biped_s46/urdf/biped_s46.urdf (robot description, URDF)
Before this commit: robot biped_s46, 46 links, 45 joints
Links:
- link leg_l6_link: geometry collision box size=0.25 0.1 0.04; visual mesh filename=package://kuavo_assets/models/biped_s46/meshes/l_foot_roll.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
- link leg_r6_link: geometry collision box size=0.25 0.1 0.04; visual mesh filename=package://kuavo_assets/models/biped_s46/meshes/r_foot_roll.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

File: src/kuavo_assets/models/biped_s46/urdf/drake/biped_v3_arm.urdf (robot description, URDF)
Before this commit: robot biped_v3_arm, 15 links, 14 joints
Links:
- removed link torso
- added link base_link, mass 26.8206; visual mesh filename=../../meshes/torso.STL
- added link zarm_l7_end_effector; collision sphere radius=0.005
- added link zarm_r7_end_effector; collision sphere radius=0.005
Joints:
- added joint zarm_l7_end_effector_joint: type fixed, parent zarm_l7_link, child zarm_l7_end_effector, origin xyz=0 -0.03 -0.17 rpy=0 0 0
- added joint zarm_r7_end_effector_joint: type fixed, parent zarm_r7_link, child zarm_r7_end_effector, origin xyz=0 0.03 -0.17 rpy=0 0 0
- joint zarm_l1_joint: origin xyz=-0.017499853 0.29269999999999996 0.4245 rpy=0 0 0 -> xyz=-0.017499853 0.29269999999999996 0.445 rpy=0 0 0; parent torso -> base_link
- joint zarm_l2_joint: limit lower=-0.349065850398866 upper=2.0943951023932 effort=50.0 velocity=19.154 -> lower=-0.349065850398866 upper=2.0943951023932 effort=50.0 velocity=8.37333333333333
- joint zarm_l3_joint: limit lower=-1.5707963267949 upper=1.5707963267949 effort=39.0 velocity=18.84 -> lower=-1.5707963267949 upper=1.5707963267949 effort=39.0 velocity=19.3633333333333
- joint zarm_l4_joint: limit lower=-2.61799387799149 upper=0.0 effort=50.0 velocity=18.84 -> lower=-2.61799387799149 upper=0.0 effort=50.0 velocity=8.37333333333333; origin xyz=0.0200000000000006 0 -0.283699999999996 rpy=0 0 0 -> xyz=0.0200000000000001 0 -0.2837 rpy=0 0 0
- joint zarm_l5_joint: limit lower=-1.5707963267949 upper=1.5707963267949 effort=12.0 velocity=21.666 -> lower=-1.5707963267949 upper=1.5707963267949 effort=12.0 velocity=7.32666666666667; origin xyz=-0.0200000000000025 0 -0.127037274261591 rpy=0 0 0 -> xyz=-0.02 0 -0.126000000138651 rpy=0 0 0
- joint zarm_l6_joint: limit lower=-1.30899693899575 upper=0.698131700797732 effort=12.0 velocity=21.666 -> lower=-1.30899693899575 upper=0.698131700797732 effort=12.0 velocity=7.32666666666667; origin xyz=0.000199999999999079 0 -0.106462725738415 rpy=0 0 0 -> xyz=0 0 -0.107499999861353 rpy=0 0 0
- joint zarm_l7_joint: limit lower=-0.698131700797732 upper=0.698131700797732 effort=12.0 velocity=21.666 -> lower=-0.698131700797732 upper=0.698131700797732 effort=12.0 velocity=7.32666666666667; origin xyz=0 0 -0.0210004653879916 rpy=0 0 0 -> xyz=0 0 -0.0209999999999992 rpy=0 0 0
- joint zarm_r1_joint: origin xyz=-0.017499853 -0.29269999999999996 0.4245 rpy=0 0 0 -> xyz=-0.017499853 -0.29269999999999996 0.445 rpy=0 0 0; parent torso -> base_link
- joint zarm_r2_joint: limit lower=-2.0943951023932 upper=0.349065850398866 effort=50.0 velocity=19.154 -> lower=-2.0943951023932 upper=0.349065850398866 effort=50.0 velocity=8.37333333333333
- joint zarm_r4_joint: limit lower=-2.61799387799149 upper=0.0 effort=50.0 velocity=18.84 -> lower=-2.61799387799149 upper=0.0 effort=50.0 velocity=8.37333333333333; origin xyz=0.0200000000000024 0 -0.2837 rpy=0 0 0 -> xyz=0.0199999999999998 0 -0.2837 rpy=0 0 0
- joint zarm_r5_joint: limit lower=-1.5707963267949 upper=1.5707963267949 effort=12.0 velocity=21.666 -> lower=-1.5707963267949 upper=1.5707963267949 effort=12.0 velocity=7.32666666666667; origin xyz=-0.0200000000000001 0 -0.127037274261587 rpy=0 0 0 -> xyz=-0.0199999999999997 0 -0.126000000138651 rpy=0 0 0
- joint zarm_r6_joint: limit lower=-0.698131700797732 upper=1.30899693899575 effort=12.0 velocity=21.666 -> lower=-0.698131700797732 upper=1.30899693899575 effort=12.0 velocity=7.32666666666667; origin xyz=0 0 -0.106462725738415 rpy=0 0 0 -> xyz=0 0 -0.107499999861352 rpy=0 0 0
- joint zarm_r7_joint: limit lower=-0.698131700797732 upper=0.698131700797732 effort=12.0 velocity=21.666 -> lower=-0.698131700797732 upper=0.698131700797732 effort=12.0 velocity=7.32666666666667; origin xyz=0 0 -0.0209999999999999 rpy=0 0 0 -> xyz=0 0 -0.0210000000000031 rpy=0 0 0

File: src/kuavo_assets/models/biped_s47/urdf/biped_s47.urdf (robot description, URDF)
Before this commit: robot biped_s47, 62 links, 61 joints
Links:
- link leg_l6_link: geometry collision box size=0.25 0.1 0.04; visual mesh filename=package://kuavo_assets/models/biped_s47/meshes/l_foot_roll.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
- link leg_r6_link: geometry collision box size=0.25 0.1 0.04; visual mesh filename=package://kuavo_assets/models/biped_s47/meshes/r_foot_roll.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

File: src/kuavo_assets/models/biped_s47/urdf/drake/biped_v3_arm.urdf (robot description, URDF)
Before this commit: robot biped_v3_arm, 31 links, 30 joints
Links:
- removed link l_b_claw_1
- removed link l_b_claw_2
- removed link l_b_claw_3
- removed link l_b_finger
- removed link l_f_claw_1
- removed link l_f_claw_2
- removed link l_f_claw_3
- removed link l_f_finger
- removed link r_b_claw_1
- removed link r_b_claw_2
- removed link r_b_claw_3
- removed link r_b_finger
- removed link r_f_claw_1
- removed link r_f_claw_2
- removed link r_f_claw_3
- removed link r_f_finger
- removed link torso
- added link base_link, mass 27.65693803; visual mesh filename=../../meshes/torso.STL
- added link zarm_l7_end_effector; collision sphere radius=0.005
- added link zarm_r7_end_effector; collision sphere radius=0.005
Joints:
- removed joint l_b_claw_1
- removed joint l_b_claw_2
- removed joint l_b_claw_3
- removed joint l_b_finger
- removed joint l_f_claw_1
- removed joint l_f_claw_2
- removed joint l_f_claw_3
- removed joint l_f_finger
- removed joint r_b_claw_1
- removed joint r_b_claw_2
- removed joint r_b_claw_3
- removed joint r_b_finger
- removed joint r_f_claw_1
- removed joint r_f_claw_2
- removed joint r_f_claw_3
- removed joint r_f_finger
- added joint zarm_l7_end_effector_joint: type fixed, parent zarm_l7_link, child zarm_l7_end_effector, origin xyz=0 -0.03 -0.17 rpy=0 0 0
- added joint zarm_r7_end_effector_joint: type fixed, parent zarm_r7_link, child zarm_r7_end_effector, origin xyz=0 0.03 -0.17 rpy=0 0 0
- joint zarm_l1_joint: parent torso -> base_link
- joint zarm_r1_joint: parent torso -> base_link

File: src/kuavo_assets/models/biped_s48/urdf/biped_s48.urdf (robot description, URDF)
Before this commit: robot biped_s48, 69 links, 68 joints
Links:
- link leg_l6_link: geometry collision box size=0.25 0.1 0.04; visual mesh filename=package://kuavo_assets/models/biped_s48/meshes/l_foot_roll.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
- link leg_r6_link: geometry collision box size=0.25 0.1 0.04; visual mesh filename=package://kuavo_assets/models/biped_s48/meshes/r_foot_roll.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

File: src/kuavo_assets/models/biped_s48/urdf/drake/biped_v3_arm.urdf (robot description, URDF)
Before this commit: robot biped_v3_arm, 15 links, 14 joints
Links:
- removed link torso
- added link base_link, mass 22.11293803; visual mesh filename=../../meshes/torso.STL
- added link zarm_l7_end_effector; collision sphere radius=0.005
- added link zarm_r7_end_effector; collision sphere radius=0.005
Joints:
- added joint zarm_l7_end_effector_joint: type fixed, parent zarm_l7_link, child zarm_l7_end_effector, origin xyz=0 -0.03 -0.17 rpy=0 0 0
- added joint zarm_r7_end_effector_joint: type fixed, parent zarm_r7_link, child zarm_r7_end_effector, origin xyz=0 0.03 -0.17 rpy=0 0 0
- joint zarm_l1_joint: parent torso -> base_link
- joint zarm_r1_joint: parent torso -> base_link

File: src/kuavo_assets/models/biped_s49/urdf/biped_s49.urdf (robot description, URDF)
Before this commit: robot biped_s49, 47 links, 46 joints
Links:
- link leg_l6_link: geometry collision box size=0.25 0.1 0.04; visual mesh filename=package://kuavo_assets/models/biped_s49/meshes/l_foot_roll.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
- link leg_r6_link: geometry collision box size=0.25 0.1 0.04; visual mesh filename=package://kuavo_assets/models/biped_s49/meshes/r_foot_roll.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

File: src/kuavo_assets/models/biped_s49/urdf/drake/biped_v3_arm.urdf (robot description, URDF)
Before this commit: robot biped_v3_arm, 15 links, 14 joints
Links:
- removed link torso
- added link base_link, mass 24.42123803; visual mesh filename=../../meshes/torso.STL
- added link zarm_l7_end_effector; collision sphere radius=0.005
- added link zarm_r7_end_effector; collision sphere radius=0.005
Joints:
- added joint zarm_l7_end_effector_joint: type fixed, parent zarm_l7_link, child zarm_l7_end_effector, origin xyz=0 -0.03 -0.17 rpy=0 0 0
- added joint zarm_r7_end_effector_joint: type fixed, parent zarm_r7_link, child zarm_r7_end_effector, origin xyz=0 0.03 -0.17 rpy=0 0 0
- joint zarm_l1_joint: parent torso -> base_link
- joint zarm_r1_joint: parent torso -> base_link
