Commit message: sync https://www.lejuhub.com/highlydynamic/kuavo-ros-control/commit/81a7517e442767dff4f55553e53c28f6aab5d7b7

File: src/kuavo_assets/models/biped_s45/urdf/drake/biped_v3_arm.urdf (robot description, URDF)
Before this commit: robot biped_s45, 17 links, 16 joints
Joints:
- joint zarm_l1_joint: limit lower=-3.14159265358979 upper=0.01 effort=100.0 velocity=41.3433333333333 -> lower=-2.4 upper=0.6 effort=100.0 velocity=41.3433333333333
- joint zarm_r1_joint: limit lower=-3.14159265358979 upper=0.01 effort=100.0 velocity=41.3433333333333 -> lower=-2.4 upper=0.6 effort=100.0 velocity=41.3433333333333

File: src/kuavo_assets/models/biped_s46/urdf/drake/biped_v3_arm.urdf (robot description, URDF)
Before this commit: robot biped_s46, 17 links, 16 joints
Joints:
- joint zarm_l1_joint: limit lower=-3.14159265358979 upper=1.5707963267949 effort=100.0 velocity=41.3433333333333 -> lower=-2.4 upper=0.6 effort=100.0 velocity=41.3433333333333
- joint zarm_r1_joint: limit lower=-3.14159265358979 upper=1.5707963267949 effort=100.0 velocity=41.3433333333333 -> lower=-2.4 upper=0.6 effort=100.0 velocity=41.3433333333333

File: src/kuavo_assets/models/biped_s47/urdf/drake/biped_v3_arm.urdf (robot description, URDF)
Before this commit: robot biped_s47, 17 links, 16 joints
Joints:
- joint zarm_l1_joint: limit lower=-3.14159265358979 upper=1.5707963267949 effort=100.0 velocity=41.3433333333333 -> lower=-2.4 upper=0.6 effort=100.0 velocity=41.3433333333333
- joint zarm_r1_joint: limit lower=-3.14159265358979 upper=1.5707963267949 effort=100.0 velocity=41.3433333333333 -> lower=-2.4 upper=0.6 effort=100.0 velocity=41.3433333333333

File: src/kuavo_assets/models/biped_s48/urdf/drake/biped_v3_arm.urdf (robot description, URDF)
Before this commit: robot biped_s48, 17 links, 16 joints
Joints:
- joint zarm_l1_joint: limit lower=-3.14159265358979 upper=1.5707963267949 effort=100.0 velocity=41.3433333333333 -> lower=-2.4 upper=0.6 effort=100.0 velocity=41.3433333333333
- joint zarm_r1_joint: limit lower=-3.14159265358979 upper=1.5707963267949 effort=100.0 velocity=41.3433333333333 -> lower=-2.4 upper=0.6 effort=100.0 velocity=41.3433333333333

File: src/kuavo_assets/models/biped_s49/urdf/drake/biped_v3_arm.urdf (robot description, URDF)
Before this commit: robot biped_s49, 17 links, 16 joints
Joints:
- joint zarm_l1_joint: limit lower=-3.14159265358979 upper=1.5707963267949 effort=100.0 velocity=41.3433333333333 -> lower=-2.4 upper=0.6 effort=100.0 velocity=41.3433333333333
- joint zarm_r1_joint: limit lower=-3.14159265358979 upper=1.5707963267949 effort=100.0 velocity=41.3433333333333 -> lower=-2.4 upper=0.6 effort=100.0 velocity=41.3433333333333
